File: Hardware/ExiFlexBoard/ExiFlexBoard.kicad_sch (KiCad schematic)
At the start: 14 parts, among them CN1 B2B-PH-K-S, CN2 ST-005-G, SW1 ERD216CSZ, U1 XIAOESP32C3, U2 PCF8574, U3 AE-TSL25721, U4 AE-S11059

Commit message: パターン配線を実施
Parts:
- added H1: MountingHole_Pad, MountingHole:MountingHole_2.2mm_M2_Pad, symbol Mechanical:MountingHole_Pad
Connections:
- net at D1.2 (A), D2.2 (A), D3.2 (A)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: now also U3.7 (VIN)
Changed lines of the file:
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@@
   (junction (at 102.87 62.23) (diameter 0) (color 0 0 0 0)
   )
+  (junction (at 90.17 55.88) (diameter 0) (color 0 0 0 0)
+  )
   (junction (at 156.21 62.23) (diameter 0) (color 0 0 0 0)
   )
@@
     (stroke (width 0) (type default) (color 0 0 0 0))
   )
+  (wire (pts (xy 90.17 55.88) (xy 95.25 55.88))
+    (stroke (width 0) (type default) (color 0 0 0 0))
+  )
   (wire (pts (xy 151.13 106.68) (xy 157.48 106.68))
     (stroke (width 0) (type default) (color 0 0 0 0))
@@
     (stroke (width 0) (type default) (color 0 0 0 0))
   )
-  (wire (pts (xy 78.74 55.88) (xy 95.25 55.88))
+  (wire (pts (xy 78.74 55.88) (xy 90.17 55.88))
     (stroke (width 0) (type default) (color 0 0 0 0))
   )
@@
   )
   (wire (pts (xy 151.13 71.12) (xy 151.13 67.31))
+    (stroke (width 0) (type default) (color 0 0 0 0))
+  )
+  (wire (pts (xy 90.17 55.88) (xy 90.17 71.12))
     (stroke (width 0) (type default) (color 0 0 0 0))
   )
@@
     (pin "9")
   )
+  (symbol (lib_id "Mechanical:MountingHole_Pad") (at 46.99 144.78 0) (unit 1)
+    (in_bom yes) (on_board yes) (fields_autoplaced)
+    (property "Reference" "H1" (id 0) (at 46.99 138.43 0))
+    (property "Value" "MountingHole_Pad" (id 1) (at 46.99 140.335 0))
+    (property "Footprint" "MountingHole:MountingHole_2.2mm_M2_Pad" (id 2) (at 46.99 144.78 0)
+      (effects (font (size 1.27 1.27)) hide)
+    )
+    (property "Datasheet" "~" (id 3) (at 46.99 144.78 0)
+      (effects (font (size 1.27 1.27)) hide)
+    )
+    (pin "1")
+  )
   (symbol (lib_id "Device:R_US") (at 130.81 109.22 180) (unit 1)
     (in_bom yes) (on_board yes) (fields_autoplaced)
@@
       (reference "D3") (unit 1) (value "LED") (footprint "LED_THT:LED_D3.0mm")
     )
+    (path "/ce6e48a6-fdde-415c-bee4-386ec389a5bc"
+      (reference "H1") (unit 1) (value "MountingHole_Pad") (footprint "MountingHole:MountingHole_2.2mm_M2_Pad")
+    )
     (path "/3de38f93-47a0-4f02-b197-c32950380b10"
